File: sensors.kicad_sch (KiCad schematic)
At the start: 0 parts

Commit message: feat: populate sensor and user interface schematic sheets; assign footprints
- Populated the Sensors schematic sheet with the following components:
    - BME280: Temperature and humidity sensor
    - Photoresistor: For measuring ambient light levels
    - Sound Sensor Section: Includes a microphone and preamplifier to amplify audio signals for microcontroller processing

- Populated the User Interface schematic sheet with:
    - Boot and reset controls for the microcontroller
    - Breakout lines for external devices:
        - One for I²C-based peripherals (e.g., OLED display)
        - One for general-purpose I/O devices

- Both the Sensors and User Interface sheets access necessary pins (e.g., I²C, GPIO, control signals) from the parent ESP32
sheet using hierarchical labels, enabling clean and modular design.

- Assigned appropriate footprints to all components.
Parts:
- added C15, C16, C17, C18: 0u1, Capacitor_SMD:C_0805_2012Metric, symbol Device:C
- added MK1: CMC-5042PF-AC, CMC-5042PF-AC:CUI_CMC-5042PF-AC, symbol CMC-5042PF-AC:CMC-5042PF-AC
- added Q1: TEMT6000X01, TEMT6000X01:TRANS_TEMT6000X01, symbol TEMT6000X01:TEMT6000X01
- added R21, R22: 4k7, Resistor_SMD:R_0805_2012Metric, symbol Device:R
- added R23, R26: 10k, Resistor_SMD:R_0805_2012Metric, symbol Device:R
- added R24: 100k, Resistor_SMD:R_0805_2012Metric, symbol Device:R
- added R25, R29: 2k, Resistor_SMD:R_0805_2012Metric, symbol Device:R
- added R27, R28: 1M, Resistor_SMD:R_0805_2012Metric, symbol Device:R
- added U2: BME280, BME280:PSON65P250X250X100-8N, symbol BME280:BME280
- added U7: MAX4466EXK, MAX4466EXK:SOT65P210X110-5N, symbol MAX4466EXK:MAX4466EXK
Connections:
- new net: C18.2, R25.2, R29.1
- new net: MK1.OUT, R27.2, R28.1, R29.2, U7.1 (IN+)
- new net +3.3V: C15.1, C16.1, R21.1, R22.1, R23.1, R25.1, R27.1, U2.2 (CSB), U2.6 (VDDIO), U2.8 (VDD), U7.5 (VCC)
- new net GND: C15.2, C16.2, C17.1, C18.1, MK1.GND, Q1.1, R24.1, R26.1, R26.2, R28.2, U2.1 (GND), U2.5 (SDO), U2.7 (GND), U7.2 (GND), U7.3 (IN-)
- new net MIC_OUT: C17.2, R24.2, U7.4 (OUT)
- new net PHOTO_C: Q1.3, R23.2
- new net SCL: R21.2, U2.4 (SCK)
- new net SDA: R22.2, U2.3 (SDI)
Other:
- note added: "BME280"
- note added: "Microphone and amplifier"
- note added: "PHOTO SENSOR"

Commit message: refactor: update label naming for net class scope resolution; set up PCB constraints
- Renamed schematic labels to follow a net class–based naming convention for
better scope resolution (e.g., labels in the SPI net class now use a SPI_ prefix).

- Configured the PCB stack-up to use a 4-layer board.

- Applied design constraints (e.g., trace width, spacing) based on the
PCB manufacturer's recommended specifications.
Connections:
- net GND: no longer C17.1, R24.1, R26.1, U7.3 (IN-)
- net MIC_OUT renamed SENSOR_MIC_OUT
- net PHOTO_C renamed SENSOR_PHOTO_C
- net SCL renamed I2C_SCL
- net SDA renamed I2C_SDA
- new net: C17.1, R24.1, R26.1, U7.3 (IN-)
Other:
- note added: "PHOTO SCMD_ENSOR"
- note removed: "PHOTO SENSOR"
- title: (none) -> Sensors
- moved on the sheet: C15, C16, R21, R22, R26, U2
